File: pcb/plytka.kicad_sch (KiCad schematic)
At the start: 55 parts, among them J1 Display, J2 Program, J3 Battery, J4 USB_C_Receptacle_USB2.0_16P, Q1 SS8050, Q2 SS8050, Q3 AO3400A, SW1 RESET, SW2 USER0, SW3 USER2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

Commit message: footprints
Parts:
- removed Q3: AO3400A, Package_TO_SOT_SMD:SOT-23, symbol Transistor_FET:AO3400A
- added C16: 10 uF, Capacitor_SMD:C_0805_2012Metric, symbol Device:C
- added D9: D_Schottky, Diode_SMD:D_SMA, symbol Device:D_Schottky
- C5: value 10u -> 4.7u
- SW2: value USER0 -> USER1
Connections:
- net 5V: now also C16.1, D9.2 (A); no longer J4.A4 (VBUS), J4.A9 (VBUS), J4.B4 (VBUS), J4.B9 (VBUS), U3.5 (VBUS)
- net BOOST_EN: now also Q1.3 (C)
- net D+: now also J4.A6 (D+), J4.B6 (D+), U3.3 (I/O2); no longer U3.4 (I/O2)
- net D-: now also J4.A7 (D-), J4.B7 (D-), U3.1 (I/O1); no longer U3.6 (I/O1)
- net DTR: now also Q2.2 (E)
- net GND: now also C16.2; no longer Q1.2 (E), Q2.2 (E)
- net RTS: now also Q1.2 (E)
- net at J4.A5 (CC1), R2.2: now also U3.6 (I/O1)
- net at J4.B5 (CC2), R3.2: now also U3.4 (I/O2)
- net GPIO0 renamed GPIO1
- net GPIO1: no longer Q1.3 (C)
- new net: D9.1 (K), J4.A4 (VBUS), J4.A9 (VBUS), J4.B4 (VBUS), J4.B9 (VBUS), U3.5 (VBUS)
Other:
- note added: "Jaki dajemy tu DEFAULT???? Nie wiadomo jak LEDy będą się zachowywać, tryb PFM może powodować lekkie migotanie, ale jest wydajniejszy niż PWM Najwyżej się zmieni to tym jumperem."
- moved on the sheet: C10, C6, C7, C8, C9, J4, LDO1, Q1, Q2, R11, R12, R2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
