File: pcb/plytka.kicad_sch (KiCad schematic)
At the start: 56 parts, among them J1 Display, J2 Program, J3 Battery, J4 USB_C_Receptacle_USB2.0_16P, Q1 SS8050, Q2 SS8050, SW1 RESET, SW2 USER1, SW3 USER2, SW4 USER3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

Commit message: Add files via upload
Parts:
- removed C16: 10 uF, Capacitor_SMD:C_0805_2012Metric, symbol Device:C
- removed D9: D_Schottky, Diode_SMD:D_SMA, symbol Device:D_Schottky
- C12: footprint (none) -> Capacitor_SMD:C_0201_0603Metric
- C13, C14, C15: footprint (none) -> Capacitor_SMD:C_1206_3216Metric
- C5: value 4.7u -> 10u
- L1: footprint (none) -> Inductor_SMD:L_1008_2520Metric
- R5: footprint (none) -> Resistor_SMD:R_0402_1005Metric
- R6, R7: footprint (none) -> Resistor_SMD:R_0603_1608Metric
- SW2: value USER1 -> USER0
Connections:
- net 5V: now also J4.A4 (VBUS), J4.A9 (VBUS), J4.B4 (VBUS), J4.B9 (VBUS), U3.5 (VBUS)
- net BOOST_EN: no longer Q1.3 (C)
- net D+: now also U3.4 (I/O2); no longer J4.A6 (D+), J4.B6 (D+), U3.3 (I/O2)
- net D-: now also U3.6 (I/O1); no longer J4.A7 (D-), J4.B7 (D-), U3.1 (I/O1)
- net DTR: no longer Q2.2 (E)
- net GND: now also Q1.2 (E), Q2.2 (E)
- net RTS: no longer Q1.2 (E)
- net at J4.A5 (CC1), R2.2: no longer U3.6 (I/O1)
- net at J4.B5 (CC2), R3.2: no longer U3.4 (I/O2)
- net GPIO1 renamed GPIO0
- net GPIO0: now also Q1.3 (C)
- new net: J4.A6 (D+), J4.B6 (D+), U3.3 (I/O2)
- new net: J4.A7 (D-), J4.B7 (D-), U3.1 (I/O1)
Other:
- note removed: "Jaki dajemy tu DEFAULT???? Nie wiadomo jak LEDy będą się zachowywać, tryb PFM może powodować lekkie migotanie, ale jest wydajniejszy niż PWM Najwyżej się zmieni to tym jumperem."
- moved on the sheet: C10, C6, C7, C8, C9, J4, LDO1, Q1, Q2, R11, R12, R2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

Commit message: miau
Parts:
- removed Q1, Q2: SS8050, Package_TO_SOT_SMD:SOT-23, symbol Transistor_BJT:SS8050
- removed R11: 10k, Resistor_SMD:R_01005_0402Metric, symbol Device:R
- removed R12: 10k, Resistor_SMD:R_0402_1005Metric, symbol Device:R
- added C16: 100n, Capacitor_SMD:C_0402_1005Metric, symbol Device:C
- added Q3, Q4: AO3400A, Package_TO_SOT_SMD:SOT-23, symbol Transistor_FET:AO3400A
Connections:
- net DTR: now also C16.1, Q3.2 (S), Q4.1 (G)
- net GPIO0: now also Q3.3 (D)
- net RESET: now also C16.2, Q4.3 (D)
- net RTS: now also Q3.1 (G), Q4.2 (S)
- net UART_RX: now also U4.8 (TXD); no longer U4.9 (RXD)
- net UART_TX: now also U4.9 (RXD); no longer U4.8 (TXD)
Other:
- note added: "LED boost converter"
- note added: "programming logic converter"
- note removed: "logic converter"
- moved on the sheet: BT1, C10, C17, C18, C5, C6, C7, C8, C9, D8, J3, J4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

Commit message: footprint
Parts:
- removed J3: Battery, Connector_PinHeader_2.54mm:PinHeader_1x02_P2.54mm_Vertical, symbol Connector:Conn_01x02_Pin
- BT1: footprint (none) -> Connector_PinHeader_2.54mm:PinHeader_1x02_P2.54mm_Vertical
- JP1: footprint (none) -> Jumper:SolderJumper-3_P1.3mm_Bridged2Bar12_Pad1.0x1.5mm
- renumbered J4 to J3
Other:
- note removed: "Battery Connector"
Changed lines of the file:
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@@
 	)
 	(rectangle
-		(start 255.27 13.97)
-		(end 281.94 55.88)
-		(stroke
-			(width 0)
-			(type default)
-		)
-		(fill
-			(type none)
-		)
-	)
-	(rectangle
 		(start 64.77 153.67)
 		(end 140.97 195.58)
@@
 		)
 	)
-	(text "Battery Connector"
-		(exclude_from_sim no)
-		(at 264.922 16.002 0)
-		(effects
-			(font
-				(size 1.27 1.27)
-			)
-		)
-	)
 	(text "2.4V max"
 		(exclude_from_sim no)
@@
 	)
 	(junction
-		(at 278.13 35.56)
-		(diameter 0)
-		(color 0 0 0 0)
-	)
-	(junction
 		(at 257.81 68.58)
 		(diameter 0)
@@
 	)
 	(junction
+		(at 102.87 138.43)
+		(diameter 0)
+		(color 0 0 0 0)
+	)
+	(junction
 		(at 213.36 38.1)
 		(diameter 0)
@@
 	(wire
 		(pts
-			(xy 278.13 35.56) (xy 278.13 38.1)
-		)
-		(stroke
-			(width 0)
-			(type default)
-		)
-	)
-	(wire
-		(pts
 			(xy 35.56 175.26) (xy 40.64 175.26)
 		)
@@
 	(wire
 		(pts
+			(xy 102.87 139.7) (xy 102.87 138.43)
+		)
+		(stroke
+			(width 0)
+			(type default)
+		)
+	)
+	(wire
+		(pts
 			(xy 161.29 120.65) (xy 160.02 120.65)
 		)
@@
 	(wire
 		(pts
-			(xy 264.16 35.56) (xy 278.13 35.56)
-		)
-		(stroke
-			(width 0)
-			(type default)
-		)
-	)
-	(wire
-		(pts
 			(xy 67.31 138.43) (xy 67.31 140.97)
 		)
@@
 	(wire
 		(pts
-			(xy 278.13 34.29) (xy 278.13 35.56)
-		)
-		(stroke
-			(width 0)
-			(type default)
-		)
-	)
-	(wire
-		(pts
 			(xy 246.38 80.01) (xy 246.38 81.28)
 		)
@@
 	(wire
 		(pts
-			(xy 264.16 38.1) (xy 266.7 38.1)
-		)
-		(stroke
-			(width 0)
-			(type default)
-		)
-	)
-	(wire
-		(pts
 			(xy 255.27 127) (xy 255.27 110.49)
 		)
@@
 		)
 	)
-	(global_label "VBAT"
-		(shape input)
-		(at 266.7 38.1 0)
-		(fields_autoplaced yes)
-		(effects
-			(font
-				(size 1.27 1.27)
-			)
-			(justify left)
-		)
-		(property "Intersheetrefs" "${INTERSHEET_REFS}"
-			(at 274.1 38.1 0)
-			(effects
-				(font
-					(size 1.27 1.27)
-				)
-				(justify left)
-				(hide yes)
-			)
-		)
-	)
 	(symbol
 		(lib_id "Device:R")
@@
 		(dnp no)
 		(fields_autoplaced yes)
-		(property "Reference" "J4"
+		(property "Reference" "J3"
 			(at 144.78 97.79 0)
 			(effects
@@
 			(project ""
 				(path "/a5474e04-ba65-41a7-9e5c-ab57fc53d54d"
-					(reference "J4")
+					(reference "J3")
 					(unit 1)
 				)
@@
 			)
 		)
-		(property "Footprint" ""
+		(property "Footprint" "Connector_PinHeader_2.54mm:PinHeader_1x02_P2.54mm_Vertical"
 			(at 102.87 130.556 90)
 			(effects
@@
 			)
 		)
-		(property "Footprint" ""
+		(property "Footprint" "Jumper:SolderJumper-3_P1.3mm_Bridged2Bar12_Pad1.0x1.5mm"
 			(at 177.8 44.45 0)
 			(effects
@@
 	)
 	(symbol
-		(lib_id "Connector:Conn_01x02_Pin")
-		(at 259.08 35.56 0)
-		(unit 1)
-		(exclude_from_sim no)
-		(in_bom yes)
-		(on_board yes)
-		(dnp no)
-		(fields_autoplaced yes)
-		(property "Reference" "J3"
-			(at 259.715 30.48 0)
-			(effects
-				(font
-					(size 1.27 1.27)
-				)
-			)
-		)
-		(property "Value" "Battery"
-			(at 259.715 33.02 0)
-			(effects
-				(font
-					(size 1.27 1.27)
-				)
-			)
-		)
-		(property "Footprint" "Connector_PinHeader_2.54mm:PinHeader_1x02_P2.54mm_Vertical"
-			(at 259.08 35.56 0)
-			(effects
-				(font
-					(size 1.27 1.27)
-				)
-				(hide yes)
-			)
-		)
-		(property "Datasheet" "~"
-			(at 259.08 35.56 0)
-			(effects
-				(font
-					(size 1.27 1.27)
-				)
-				(hide yes)
-			)
-		)
-		(property "Description" "Generic connector, single row, 01x02, script generated"
-			(at 259.08 35.56 0)
-			(effects
-				(font
-					(size 1.27 1.27)
-				)
-				(hide yes)
-			)
-		)
-		(pin "2"
-		)
-		(pin "1"
-		)
-		(instances
-			(project "plytka"
-				(path "/a5474e04-ba65-41a7-9e5c-ab57fc53d54d"
-					(reference "J3")
-					(unit 1)
-				)
-			)
-		)
-	)
-	(symbol
 		(lib_id "library:TP4054")
 		(at 67.31 118.11 0)
@@
 	)
 	(symbol
-		(lib_id "power:GND")
-		(at 278.13 38.1 0)
-		(unit 1)
-		(exclude_from_sim no)
-		(in_bom yes)
-		(on_board yes)
-		(dnp no)
-		(property "Reference" "#PWR02"
-			(at 278.13 44.45 0)
-			(effects
-				(font
-					(size 1.27 1.27)
-				)
-				(hide yes)
-			)
-		)
-		(property "Value" "GND"
-			(at 278.13 42.164 0)
-			(effects
-				(font
-					(size 1.27 1.27)
-				)
-			)
-		)
-		(property "Footprint" ""
-			(at 278.13 38.1 0)
-			(effects
-				(font
-					(size 1.27 1.27)
-				)
-				(hide yes)
-			)
-		)
-		(property "Datasheet" ""
-			(at 278.13 38.1 0)
-			(effects
-				(font
-					(size 1.27 1.27)
-				)
-				(hide yes)
-			)
-		)
-		(property "Description" "Power symbol creates a global label with name \"GND\" , ground"
-			(at 278.13 38.1 0)
-			(effects
-				(font
-					(size 1.27 1.27)
-				)
-				(hide yes)
-			)
-		)
-		(pin "1"
-		)
-		(instances
-			(project "plytka"
-				(path "/a5474e04-ba65-41a7-9e5c-ab57fc53d54d"
-					(reference "#PWR02")
-					(unit 1)
-				)
-			)
-		)
-	)
-	(symbol
 		(lib_id "Device:R")
 		(at 22.86 180.34 0)
@@
 	(symbol
 		(lib_id "power:PWR_FLAG")
-		(at 278.13 34.29 0)
+		(at 102.87 139.7 180)
 		(unit 1)
 		(exclude_from_sim no)
@@
 		(dnp no)
 		(property "Reference" "#FLG01"
-			(at 278.13 32.385 0)
+			(at 102.87 141.605 0)
 			(effects
 				(font
@@
 		)
 		(property "Value" "GND"
-			(at 278.13 30.226 0)
+			(at 102.87 143.764 0)
 			(effects
 				(font
@@
 		)
 		(property "Footprint" ""
-			(at 278.13 34.29 0)
+			(at 102.87 139.7 0)
 			(effects
 				(font
@@
 		)
 		(property "Datasheet" "~"
-			(at 278.13 34.29 0)
+			(at 102.87 139.7 0)
 			(effects
 				(font
@@
 		)
 		(property "Description" "Special symbol for telling ERC where power comes from"
-			(at 278.13 34.29 0)
+			(at 102.87 139.7 0)
 			(effects
 				(font

Commit message: lcsc
Parts:
- C1, C16, C17, C18, C2, C3, C4: LCSC (none) -> C1525
- C10, C11, C8: footprint Capacitor_SMD:C_0201_0603Metric -> Capacitor_SMD:C_0402_1005Metric; LCSC (none) -> C1525
- C12, C5, C6, C7, C9: footprint Capacitor_SMD:C_0201_0603Metric -> Capacitor_SMD:C_0402_1005Metric; LCSC (none) -> C15525
- C13, C14, C15: footprint Capacitor_SMD:C_1206_3216Metric -> Capacitor_SMD:C_0805_2012Metric; LCSC (none) -> C45783
- D1, D2, D3, D4, D5, D6, D7: LCSC (none) -> C2761795
- J3: LCSC (none) -> C9900016516
- L1: LCSC (none) -> C2849428
- R1: value 2.5K -> 2.4K; LCSC (none) -> C22940
- R10, R9: footprint Resistor_SMD:R_0201_0603Metric -> Resistor_SMD:R_0805_2012Metric; LCSC (none) -> C17514
- R2, R3: LCSC (none) -> C23186
- R5: footprint Resistor_SMD:R_0402_1005Metric -> Resistor_SMD:R_0805_2012Metric; LCSC (none) -> C17710
- R6: LCSC (none) -> C13281
- R7: footprint Resistor_SMD:R_0603_1608Metric -> Capacitor_SMD:C_0201_0603Metric; LCSC (none) -> C25803
- SW1, SW2, SW3, SW4: footprint Button_Switch_SMD:SW_SPST_Omron_B3FS-100xP -> Button_Switch_THT:SW_TH_Tactile_Omron_B3F-100x
- U3: LCSC (none) -> C2827693
- U4: LCSC (none) -> C2977777

Commit message: almost finish pcb
Parts:
- removed J2: Program, Connector_PinHeader_2.54mm:PinHeader_1x04_P2.54mm_Vertical, symbol Connector:Conn_01x04_Pin
- C1, C10, C11, C16, C17, C18, C2, C3, C4, C8: LCSC C1525 -> (none)
- C12, C5, C6, C7, C9: footprint Capacitor_SMD:C_0402_1005Metric -> Capacitor_SMD:C_0603_1608Metric; LCSC C15525 -> (none)
- C13, C14, C15: footprint Capacitor_SMD:C_0805_2012Metric -> Capacitor_SMD:C_0603_1608Metric; LCSC C45783 -> (none)
- D1, D2, D3, D4, D5, D6, D7: LCSC C2761795 -> (none)
- J3: LCSC C9900016516 -> (none)
- L1: LCSC C2849428 -> (none)
- R1: value 2.4K -> 2.5K; LCSC C22940 -> (none)
- R10, R9: footprint Resistor_SMD:R_0805_2012Metric -> Resistor_SMD:R_0201_0603Metric; LCSC C17514 -> (none)
- R2, R3: LCSC C23186 -> (none)
- R5: footprint Resistor_SMD:R_0805_2012Metric -> Resistor_SMD:R_0402_1005Metric; LCSC C17710 -> (none)
- R6: LCSC C13281 -> (none)
- R7: footprint Capacitor_SMD:C_0201_0603Metric -> Resistor_SMD:R_0603_1608Metric; LCSC C25803 -> (none)
- SW1: renamed from SW2; footprint Button_Switch_THT:SW_TH_Tactile_Omron_B3F-100x -> Button_Switch_SMD:SW_Push_1P1T-MP_NO_Horizontal_Alps_SKRTLAE010
- SW2: renamed from SW3; value USER2 -> USER6; footprint Button_Switch_THT:SW_TH_Tactile_Omron_B3F-100x -> Button_Switch_SMD:SW_Push_1P1T-MP_NO_Horizontal_Alps_SKRTLAE010
- SW3: renamed from SW4; value USER3 -> USER7; footprint Button_Switch_THT:SW_TH_Tactile_Omron_B3F-100x -> Button_Switch_SMD:SW_Push_1P1T-MP_NO_Horizontal_Alps_SKRTLAE010
- SW4: renamed from SW1; footprint Button_Switch_THT:SW_TH_Tactile_Omron_B3F-100x -> Button_Switch_SMD:SW_Push_1P1T-MP_NO_Horizontal_Alps_SKRTLAE010
- U3: LCSC C2827693 -> (none)
- U4: LCSC C2977777 -> (none)
Connections:
- net BAT_LVL: now also HTCC-AM1.10 (ADC)
- net D+: now also U3.6 (I/O1); no longer U3.4 (I/O2)
- net D-: now also U3.4 (I/O2); no longer U3.6 (I/O1)
- net at J3.A6 (D+), J3.B6 (D+): now also U3.1 (I/O1); no longer U3.3 (I/O2)
- net at J3.A7 (D-), J3.B7 (D-): now also U3.3 (I/O2); no longer U3.1 (I/O1)
- no-connect marks 12 -> 11
Other:
- note removed: "Programming Connector"
- moved on the sheet: C10, C7, C8, C9, LDO1

Commit message: lcsc
Parts:
- added R4: 220k, Resistor_SMD:R_0603_1608Metric, symbol Device:R
- C1, C10, C11, C16, C17, C18, C2, C3, C4, C8: LCSC (none) -> C307331
- C12, C5, C6, C7, C9: LCSC (none) -> C19702
- C13, C14, C15: LCSC (none) -> C59461
- D1, D2, D3, D4, D5, D6, D7: LCSC (none) -> C2761795
- D8: LCSC (none) -> C7420331
- L1: LCSC (none) -> C2849428
- LDO1: LCSC (none) -> C5357206
- Q3, Q4: LCSC (none) -> C1525
- R1: value 2.5K -> 2.4k; footprint Resistor_SMD:R_0201_0603Metric -> Resistor_SMD:R_0603_1608Metric; LCSC (none) -> C22940
- R10, R9: footprint Resistor_SMD:R_0201_0603Metric -> Resistor_SMD:R_0402_1005Metric; LCSC (none) -> C26083
- R2: value 5.1 k -> 5.1k; LCSC (none) -> C23186
- R3: LCSC (none) -> C23186
- R5: LCSC (none) -> C25117
- R6: value 732k -> 510k; LCSC (none) -> C23192
- R7: LCSC (none) -> C23192
- U1: LCSC (none) -> C915088
- U2: LCSC (none) -> C32574
- U3: LCSC (none) -> C2827693
- U4: LCSC (none) -> C968586
Connections:
- net at R7.1, U1.4 (FB): now also R4.2; no longer R6.2
- new net: R4.1, R6.2
Other:
- note added: "417mA charge current (0.83C)"
- note removed: "250mA charge current (0.5C)"
- moved on the sheet: R6

Commit message: final final final??
Parts:
- D1, D2, D3, D4, D5, D6, D7: LCSC C2761795 -> C48586674
- J3: LCSC (none) -> C2988369
- Q1: renamed from Q3; LCSC C1525 -> C20917
- Q2: renamed from Q4; LCSC C1525 -> C20917
- R7: LCSC C23192 -> C25803
- SW1: value USER0 -> TS24CA; footprint Button_Switch_SMD:SW_Push_1P1T-MP_NO_Horizontal_Alps_SKRTLAE010 -> Library:SW_TS31-46-35-BK-B-160-RA-SMT-TR; LCSC (none) -> C393942
- SW2: value USER6 -> TS24CA; footprint Button_Switch_SMD:SW_Push_1P1T-MP_NO_Horizontal_Alps_SKRTLAE010 -> Library:SW_TS31-46-35-BK-B-160-RA-SMT-TR; LCSC (none) -> C393942
- SW3: value USER7 -> TS24CA; footprint Button_Switch_SMD:SW_Push_1P1T-MP_NO_Horizontal_Alps_SKRTLAE010 -> Library:SW_TS31-46-35-BK-B-160-RA-SMT-TR; LCSC (none) -> C393942
- SW4: value RESET -> TS24CA; footprint Button_Switch_SMD:SW_Push_1P1T-MP_NO_Horizontal_Alps_SKRTLAE010 -> Library:SW_TS31-46-35-BK-B-160-RA-SMT-TR; LCSC (none) -> C393942
