File: pcb/plytka.kicad_pcb (KiCad board)
At the start: 2 copper layers, 29.2 x 77.9 mm, 58 parts, among them J1 Display, J3 USB_C_Receptacle_USB2.0_16P, Q3 AO3400A, Q4 AO3400A, SW1 USER0, SW2 USER6, SW3 USER7, SW4 RESET, U1 TPS61022, U2 TP4054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

Commit message: dopiesczenie:)
Routing:
- net 3V3: track 95.0 -> 95.6 mm
- net 5V: track 20.4 -> 20.9 mm, vias 3 -> 4
- net GND: track 110.2 -> 110.5 mm, vias 22 -> 86

Commit message: nonchalant zaokronglenia
Routing:
- net GND: track 110.5 -> 108.6 mm, vias 86 -> 85
- net RESET: track 52.5 -> 51.5 mm
- net UART_RX: track 61.1 -> 60.2 mm
- net GPIO0: track 37.5 -> 36.6 mm
- net UART_TX: track 61.4 -> 60.6 mm
- net BOOST_EN: track 60.9 -> 60.1 mm
- net DTR: track 68.5 -> 67.8 mm
- net Net-(D8-K): track 24.1 -> 23.5 mm
- net RTS: track 62.5 -> 62.0 mm
- net Net-(J3-D--PadA7): track 13.3 -> 12.7 mm

Commit message: final final final??
Parts:
- SW1: value USER0 -> TS24CA; footprint Button_Switch_SMD:SW_Push_1P1T-MP_NO_Horizontal_Alps_SKRTLAE010 -> Library:SW_TS31-46-35-BK-B-160-RA-SMT-TR
- SW2: value USER6 -> TS24CA; footprint Button_Switch_SMD:SW_Push_1P1T-MP_NO_Horizontal_Alps_SKRTLAE010 -> Library:SW_TS31-46-35-BK-B-160-RA-SMT-TR
- SW3: value USER7 -> TS24CA; footprint Button_Switch_SMD:SW_Push_1P1T-MP_NO_Horizontal_Alps_SKRTLAE010 -> Library:SW_TS31-46-35-BK-B-160-RA-SMT-TR
- SW4: value RESET -> TS24CA; footprint Button_Switch_SMD:SW_Push_1P1T-MP_NO_Horizontal_Alps_SKRTLAE010 -> Library:SW_TS31-46-35-BK-B-160-RA-SMT-TR
- renumbered Q3 to Q1, Q4 to Q2
Routing:
- net GND: track 108.6 -> 83.8 mm
- net (no net): track 0.00 -> 17.0 mm
- net GPIO7: track 22.8 -> 20.9 mm
- net RESET: track 51.5 -> 50.3 mm
- net GPIO6: track 17.3 -> 16.3 mm
- net Net-(J3-D--PadA7): track 12.7 -> 12.0 mm
- net VBAT: track 44.9 -> 45.6 mm
- net BAT_LVL: track 57.1 -> 57.7 mm
- net GPIO0: track 36.6 -> 37.1 mm
Other:
- outline, holes or cut-outs redrawn
